File: KiCAD/KNTTRL_ControlBoard/KNTTRL_ControlBoard.kicad_pcb (KiCad board)
At the start: 2 copper layers, 149.9 x 41.7 mm, 33 parts, among them J1 Conn_01x07, J2 Conn_01x04, J3 Conn_01x02, Q1 2N7000, Q2 2N7000, Q3 2N7000, Q4 2N7000, Q5 2N7000, U1 PC817, U2 PC817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

Commit message: update KiCAD files
Parts:
- C103: value 100nF -> 1uF; footprint Capacitor_THT:C_Disc_D5.0mm_W2.5mm_P2.50mm -> Capacitor_THT:CP_Radial_D5.0mm_P2.50mm
- moved C103 2.54 mm to (142.2, 86.4), turned to 90 degrees
Connections:
- C103 pad 1: GND -> HEATER_R
- C103 pad 2: HEATER_R -> GND
