File: KiCAD/KNTTRL_ControlBoard/KNTTRL_ControlBoard.kicad_sch (KiCad schematic)
At the start: 33 parts, among them J1 Conn_01x07, J2 Conn_01x04, J3 Conn_01x02, Q1 2N7000, Q2 2N7000, Q3 2N7000, Q4 2N7000, Q5 2N7000, U1 PC817, U2 PC817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

Commit message: update KiCAD files
Parts:
- C103: value 100nF -> 1uF; footprint Capacitor_THT:C_Disc_D5.0mm_W2.5mm_P2.50mm -> Capacitor_THT:CP_Radial_D5.0mm_P2.50mm; symbol Device:C -> Device:C_Polarized
Connections:
- net GND: now also C103.2; no longer C103.1
- net HEATER_R: now also C103.1; no longer C103.2
Changed lines of the file:
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@@
 	(wire
 		(pts
-			(xy 170.18 130.81) (xy 170.18 132.08)
-		)
-		(stroke
-			(width 0)
-			(type default)
-		)
-	)
-	(wire
-		(pts
 			(xy 182.88 99.06) (xy 82.55 99.06)
 		)
@@
 	(wire
 		(pts
+			(xy 170.18 114.3) (xy 170.18 119.38)
+		)
+		(stroke
+			(width 0)
+			(type default)
+		)
+	)
+	(wire
+		(pts
 			(xy 99.06 171.45) (xy 99.06 168.91)
 		)
@@
 	(wire
 		(pts
+			(xy 170.18 127) (xy 170.18 132.08)
+		)
+		(stroke
+			(width 0)
+			(type default)
+		)
+	)
+	(wire
+		(pts
 			(xy 228.6 85.09) (xy 228.6 90.17)
 		)
@@
 	(global_label "GND"
 		(shape input)
-		(at 170.18 123.19 90)
+		(at 170.18 114.3 90)
 		(fields_autoplaced yes)
 		(effects
@@
 		)
 		(property "Intersheetrefs" "${INTERSHEET_REFS}"
-			(at 170.18 116.3343 90)
+			(at 170.18 107.4443 90)
 			(effects
 				(font
@@
 	)
 	(symbol
-		(lib_id "Device:C")
-		(at 170.18 127 0)
+		(lib_id "Device:C_Polarized")
+		(at 170.18 123.19 180)
 		(unit 1)
 		(exclude_from_sim no)
@@
 		(fields_autoplaced yes)
 		(property "Reference" "C103"
-			(at 173.99 125.7299 0)
+			(at 173.99 122.8089 0)
 			(effects
 				(font
 					(size 1.27 1.27)
 				)
-				(justify left)
+				(justify right)
 			)
 		)
-		(property "Value" "100nF"
-			(at 173.99 128.2699 0)
+		(property "Value" "1uF"
+			(at 173.99 125.3489 0)
 			(effects
 				(font
 					(size 1.27 1.27)
 				)
-				(justify left)
+				(justify right)
 			)
 		)
-		(property "Footprint" "Capacitor_THT:C_Disc_D5.0mm_W2.5mm_P2.50mm"
-			(at 171.1452 130.81 0)
+		(property "Footprint" "Capacitor_THT:CP_Radial_D5.0mm_P2.50mm"
+			(at 169.2148 119.38 0)
 			(effects
 				(font
@@
 		)
 		(property "Datasheet" "~"
-			(at 170.18 127 0)
+			(at 170.18 123.19 0)
 			(effects
 				(font
@@
 			)
 		)
-		(property "Description" "Unpolarized capacitor"
-			(at 170.18 127 0)
+		(property "Description" "Polarized capacitor"
+			(at 170.18 123.19 0)
 			(effects
 				(font
